File: src/src.kicad_sch (KiCad schematic)
At the start: 0 parts

Commit message: Completed the schematic!
Parts:
- added C1: 10uF, symbol Device:C_US
- added C2: 10nF, symbol Device:C
- added D1: LED, symbol Device:LED
- added J1: 5V DC, symbol Connector:Jack-DC
- added R1: 1k, symbol Device:R
- added R2: 100k, symbol Device:R
- added R3: 220, symbol Device:R
- added U1: NE555P, Package_DIP:DIP-8_W7.62mm, symbol Timer:NE555P
Connections:
- new net: C2.1, U1.5 (CONT)
- new net: R1.1, R2.1, U1.7 (DISCH)
- new net: C1.1, R2.2, U1.2 (TRIG), U1.6 (THRES)
- new net: J1.1, R1.2, U1.4 (~{RST}), U1.8 (VCC)
- new net: D1.2 (A), R3.2
- new net: R3.1, U1.3 (OUT)
- new net GND: C1.2, C2.2, D1.1 (K), J1.2, U1.1 (GND)

Commit message: Comlpeted the routing and DRC. All checks passed!
This board is now ready for production hehe.
Parts:
- C1: footprint (none) -> Capacitor_THT:CP_Radial_D5.0mm_P2.00mm
- C2: footprint (none) -> Capacitor_THT:C_Disc_D5.0mm_W2.5mm_P5.00mm
- D1: footprint (none) -> LED_THT:LED_D5.0mm
- J1: footprint (none) -> Connector_BarrelJack:BarrelJack_Horizontal
- R1, R2, R3: footprint (none) -> Resistor_THT:R_Axial_DIN0207_L6.3mm_D2.5mm_P10.16mm_Horizontal
Changed lines of the file:
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@@
 			)
 		)
-		(property "Footprint" ""
+		(property "Footprint" "Capacitor_THT:C_Disc_D5.0mm_W2.5mm_P5.00mm"
 			(at 169.2148 85.09 0)
 			(hide yes)
@@
 			)
 		)
-		(property "Footprint" ""
+		(property "Footprint" "Resistor_THT:R_Axial_DIN0207_L6.3mm_D2.5mm_P10.16mm_Horizontal"
 			(at 137.16 102.362 90)
 			(hide yes)
@@
 			)
 		)
-		(property "Footprint" ""
+		(property "Footprint" "Connector_BarrelJack:BarrelJack_Horizontal"
 			(at 159.004 74.93 0)
 			(hide yes)
@@
 			)
 		)
-		(property "Footprint" ""
+		(property "Footprint" "LED_THT:LED_D5.0mm"
 			(at 205.74 113.03 0)
 			(hide yes)
@@
 			)
 		)
-		(property "Footprint" ""
+		(property "Footprint" "Resistor_THT:R_Axial_DIN0207_L6.3mm_D2.5mm_P10.16mm_Horizontal"
 			(at 196.85 114.808 90)
 			(hide yes)
@@
 			)
 		)
-		(property "Footprint" ""
+		(property "Footprint" "Capacitor_THT:CP_Radial_D5.0mm_P2.00mm"
 			(at 149.86 119.38 0)
 			(hide yes)
@@
 			)
 		)
-		(property "Footprint" ""
+		(property "Footprint" "Resistor_THT:R_Axial_DIN0207_L6.3mm_D2.5mm_P10.16mm_Horizontal"
 			(at 128.27 104.902 90)
 			(hide yes)
